Commit message: xml整理

File: floating_manipulator.xacro (robot description, xacro)
@@ -1,23 +1,4 @@
 <?xml version="1.0"?>
-<mujoco model="adeos_ii_simulation" xmlns:xacro="http://www.ros.org/wiki/xacro">
-    <!--
-        ADEOS II (Midori II) Satellite Model
-        質量
-        燃料135kg http://www.astronautix.com/a/adeos.html
-        太陽電池171kg https://doi.org/10.1109/PVSC.1996.564010
-    -->
-    <!--
-        TODOLIST:
-        - 取付位置の偏心の再現？
-    -->
-    <!-- 変数の定義 -->
-    <!-- 衛星本体のサイズ (半分の長さ) -->
-    <xacro:property name="satellite_size_x" value="6" />
-    <xacro:property name="satellite_size_y" value="4" />
-    <xacro:property name="satellite_size_z" value="4" />
-    <!-- ソーラーパネルのサイズ (半分の長さ) -->
-    <xacro:property name="solar_array_size_x" value="0.20" />
-    <xacro:property name="solar_array_size_y" value="26" />
-    <xacro:property name="solar_array_size_z" value="2.6" />
+<mujoco model="floating_manipulator" xmlns:xacro="http://www.ros.org/wiki/xacro">
     <option gravity="0 0 0" timestep="0.01" />
     <visual>
@@ -29,17 +10,29 @@
         <light pos="0 0 100" dir="0 0 -1" diffuse="0.8 0.8 0.8" />
         <light pos="100 100 100" dir="-1 -1 -1" diffuse="0.5 0.5 0.5" />
-        <body name="satellite" pos="0 80 0">
+        <body name="adeos2" pos="0 80 0">
+            <!--
+                ADEOS II (Midori II) 4x4x6[m] 3.7[t] https://www.jaxa.jp/projects/sat/adeos2/index_j.html
+                太陽電池171kg 2.6x26[m] 171[kg]  https://doi.org/10.1109/PVSC.1996.564010
+                ADEOS1 燃料135kg? http://www.astronautix.com/a/adeos.html
+            -->
+            <!-- properties -->
+            <xacro:property name="adeos2_base_size_x" value="6" />
+            <xacro:property name="adeos2_base_size_y" value="4" />
+            <xacro:property name="adeos2_base_size_z" value="4" />
+            <xacro:property name="adeos2_solar_size_x" value="0.20" />
+            <xacro:property name="adeos2_solar_size_y" value="26" />
+            <xacro:property name="adeos2_solar_size_z" value="2.6" />
             <freejoint />
             <!-- Main satellite body -->
             <geom type="box"
-                size="${satellite_size_x/2} ${satellite_size_y/2} ${satellite_size_z/2}"
+                size="${adeos2_base_size_x/2} ${adeos2_base_size_y/2} ${adeos2_base_size_z/2}"
                 rgba="0.7 0.7 0.7 1" mass="3529" />
             <!-- Single large solar array paddle -->
-            <body name="solar_array" pos="2 ${(satellite_size_y + solar_array_size_y)/2} 0">
+            <body name="solar_array" pos="2 ${(adeos2_base_size_y + adeos2_solar_size_y)/2} 0">
+                <!-- 適当な偏心 -->
                 <geom type="box"
-                    size="${solar_array_size_x/2} ${solar_array_size_y/2} ${solar_array_size_z/2}"
+                    size="${adeos2_solar_size_x/2} ${adeos2_solar_size_y/2} ${adeos2_solar_size_z/2}"
                     rgba="0.1 0.1 0.5 1" mass="171" />
             </body>
-            <camera name="track" pos="40 10 0" xyaxes="0 1 0 0 0 1" mode="track" />
         </body>
     </worldbody>

Commit message: xacroって配列使えるんだ

File: floating_manipulator.xacro (robot description, xacro)
@@ -17,22 +17,18 @@
             -->
             <!-- properties -->
-            <xacro:property name="adeos2_base_size_x" value="6" />
-            <xacro:property name="adeos2_base_size_y" value="4" />
-            <xacro:property name="adeos2_base_size_z" value="4" />
-            <xacro:property name="adeos2_solar_size_x" value="0.20" />
-            <xacro:property name="adeos2_solar_size_y" value="26" />
-            <xacro:property name="adeos2_solar_size_z" value="2.6" />
+            <xacro:property name="adeos2_base_size" value="${[6, 4, 4]}" />
+            <xacro:property name="adeos2_solar_size" value="${[0.20, 26, 2.6]}" />
             <freejoint />
             <!-- Main satellite body -->
             <body name="base" pos="0 0 0">
                 <geom type="box"
-                    size="${adeos2_base_size_x/2} ${adeos2_base_size_y/2} ${adeos2_base_size_z/2}"
+                    size="${adeos2_base_size[0]/2} ${adeos2_base_size[1]/2} ${adeos2_base_size[2]/2}"
                     rgba="0.7 0.7 0.7 1" mass="3529" />
             </body>
             <!-- Single large solar array paddle -->
-            <body name="solar_array" pos="2 ${(adeos2_base_size_y + adeos2_solar_size_y)/2} 0">
+            <body name="solar_array" pos="2 ${(adeos2_base_size[1] + adeos2_solar_size[1])/2} 0">
                 <!-- 適当な偏心 -->
                 <geom type="box"
-                    size="${adeos2_solar_size_x/2} ${adeos2_solar_size_y/2} ${adeos2_solar_size_z/2}"
+                    size="${adeos2_solar_size[0]/2} ${adeos2_solar_size[1]/2} ${adeos2_solar_size[2]/2}"
                     rgba="0.1 0.1 0.5 1" mass="171" />
             </body>
@@ -40,5 +36,5 @@
     </worldbody>
     <keyframe>
-        <key name="stationary" qpos="0 0 0 1 0 0 0" qvel="0 0 0 0 0 0" />
+        <key name="stationary" qpos="0 0 0 1 0 0 0" qvel="0 0 0 0 3 0" />
     </keyframe>
 </mujoco>
