Commit message: 出典とかを追記

File: test_sat.xacro (robot description, xacro)
@@ -1,8 +1,4 @@
 <?xml version="1.0"?>
 <mujoco model="ets7" xmlns:xacro="http://www.ros.org/wiki/xacro">
-    <!--
-  This model was converted from the MATLAB SpaceDyn parameters provided in
-  ets7_linkparam.m and ets7_fig3d.m.
-  -->
     <compiler angle="radian" eulerseq="XYZ" />
     <option timestep="0.001" gravity="0 0 0">
@@ -15,14 +11,23 @@
         <camera name="overview" pos="3 -3 2" xyaxes="0.707 0.707 0 -0.408 0.408 0.816" />
         <light diffuse=".5 .5 .5" pos="0 0 3" dir="0 0 -1" />
+        <!-- variables for ChaserSatellite base. -->
+        <!-- Source:ADRAS-J https://www.mext.go.jp/content/20241122-mxt_uchukai01-000038822_2.pdf -->
+        <xacro:property name="cs_base_size" value="${[0.83, 1.2, 0.81]}" />
+        <xacro:property name="cs_base_mass" value="${150}" />
+        <!-- variables for ChaserSatellite links -->
+        <!-- Source:ETS7 https://doi.org/10.1177/0278364903022005003-->
+        <xacro:property name="cs_link_len" value="${[0.350, 0.870, 0.630, 0.275, 0.277, 0.532]}" />
+        <xacro:property name="cs_link_mass" value="${[35.0, 22.5, 21.9, 16.5, 26.0, 18.5]}" />
+        <xacro:property name="cs_link_dir"
+            value="${['0 0 1', '0 0 1', '0 0 1', '0 0 1', '0 0 1', '0 0 1']}" />
         <!-- ChaserSatellite -->
         <body name="cs_base" pos="0 0 0">
             <freejoint name="root" />
-            <xacro:property name="cs_base_size" value="${[0.83, 1.2, 0.81]}" />
             <geom name="base_geom" type="box"
                 size="${cs_base_size[0]/2} ${cs_base_size[1]/2} ${cs_base_size[2]/2}"
-                rgba="0.6 0.8 1.0 1" mass="150" />
+                rgba="0.6 0.8 1.0 1" mass="${cs_base_mass}" />
             <!-- Link 1 -->
             <body name="link1" pos="0.6 0 0" euler="0 0 0">
-                <joint name="joint1" type="hinge" axis="0 0 1" pos="0 0 0" />
+                <joint name="joint1" type="hinge" axis="${cs_link_dir[0]}" pos="0 0 0" />
                 <geom name="link1_geom" type="box" size="0.05 0.05 0.175" pos="0 0 -0.175"
                     rgba="0.6 0.8 1.0 1" mass="35.0" />

Commit message: リンクの向き以外多分合った

File: test_sat.xacro (robot description, xacro)
@@ -8,4 +8,8 @@
         <global offwidth="1280" offheight="720" />
     </visual>
+    <default>
+        <joint type="hinge" />
+        <geom type="capsule" size="0.05" rgba="0.6 0.8 1.0 1" />
+    </default>
     <worldbody>
         <camera name="overview" pos="3 -3 2" xyaxes="0.707 0.707 0 -0.408 0.408 0.816" />
@@ -19,6 +23,6 @@
         <xacro:property name="cs_link_len" value="${[0.350, 0.870, 0.630, 0.275, 0.277, 0.532]}" />
         <xacro:property name="cs_link_mass" value="${[35.0, 22.5, 21.9, 16.5, 26.0, 18.5]}" />
-        <xacro:property name="cs_link_dir"
-            value="${['0 0 1', '0 0 1', '0 0 1', '0 0 1', '0 0 1', '0 0 1']}" />
+        <xacro:property name="cs_link_axis"
+            value="${['0 0 1', '0 1 0', '0 1 0', '0 1 0', '0 0 1', '0 1 0']}" />
         <!-- ChaserSatellite -->
         <body name="cs_base" pos="0 0 0">
@@ -28,35 +32,32 @@
                 rgba="0.6 0.8 1.0 1" mass="${cs_base_mass}" />
             <!-- Link 1 -->
-            <body name="link1" pos="0.6 0 0" euler="0 0 0">
-                <joint name="joint1" type="hinge" axis="${cs_link_dir[0]}" pos="0 0 0" />
-                <geom name="link1_geom" type="box" size="0.05 0.05 0.175" pos="0 0 -0.175"
-                    rgba="0.6 0.8 1.0 1" mass="35.0" />
+            <body name="link0" pos="0.6 0 0">
+                <joint name="joint0" axis="${cs_link_axis[0]}" />
+                <geom fromto="0 0 0 0 0 -${cs_link_len[0]}" mass="${cs_link_mass[0]}" />
                 <!-- Link 2 -->
-                <body name="link2" pos="0.28 0 0.175" euler="0 1.570796 3.141593">
-                    <joint name="joint2" type="hinge" axis="1 0 0" pos="0 0 0" />
-                    <geom name="link2_geom" type="box" size="0.435 0.05 0.05" pos="-0.435 0 0"
-                        rgba="0.6 0.8 1.0 1" mass="22.5" />
+                <body name="link1" pos="0 0 -${cs_link_len[0]}">
+                    <joint name="joint1" axis="${cs_link_axis[1]}" />
+                    <geom fromto="0 0 0 ${cs_link_len[1]} 0 0" mass="${cs_link_mass[1]}" />
                     <!-- Link 3 -->
-                    <body name="link3" pos="0.435 0 0" euler="0 3.141593 1.570796">
-                        <joint name="joint3" type="hinge" axis="1 0 0" pos="0 0 0" />
-                        <geom name="link3_geom" type="box" size="0.315 0.05 0.05" pos="-0.315 0 0"
-                            rgba="0.6 0.8 1.0 1" mass="21.9" />
+                    <body name="link2" pos="${cs_link_len[1]} 0 0">
+                        <joint name="joint2" axis="${cs_link_axis[2]}" />
+                        <geom fromto="0 0 0 0 0 -${cs_link_len[2]}" mass="${cs_link_mass[2]}" />
                         <!-- Link 4 -->
-                        <body name="link4" pos="0.315 0 0" euler="0 1.570796 3.141593">
-                            <joint name="joint4" type="hinge" axis="1 0 0" pos="0 0 0" />
-                            <geom name="link4_geom" type="box" size="0.1375 0.05 0.05"
-                                pos="-0.1375 0 0" rgba="0.6 0.8 1.0 1" mass="16.5" />
+                        <body name="link3" pos="0 0 -${cs_link_len[2]}">
+                            <joint name="joint3" axis="${cs_link_axis[3]}" />
+                            <geom fromto="0 0 0 ${cs_link_len[3]} 0 0" mass="${cs_link_mass[3]}" />
                             <!-- Link 5 -->
-                            <body name="link5" pos="0.1375 0 0" euler="0 1.570796 -1.570796">
-                                <joint name="joint5" type="hinge" axis="1 0 0" pos="0 0 0" />
-                                <geom name="link5_geom" type="box" size="0.1385 0.05 0.05"
-                                    pos="-0.1385 0 0" rgba="0.6 0.8 1.0 1" mass="26.0" />
+                            <body name="link4" pos="${cs_link_len[3]} 0 0">
+                                <joint name="joint4" axis="${cs_link_axis[4]}" />
+                                <geom fromto="0 0 0 ${cs_link_len[4]} 0 0" mass="${cs_link_mass[4]}" />
                                 <!-- Link 6 -->
-                                <body name="link6" pos="0.1385 0 0" euler="0 1.570796 -1.570796">
-                                    <joint name="joint6" type="hinge" axis="1 0 0" pos="0 0 0" />
-                                    <geom name="link6_geom" type="box" size="0.266 0.05 0.05"
-                                        pos="-0.266 0 0" rgba="0.6 0.8 1.0 1" mass="18.5" />
+                                <body name="link5" pos="${cs_link_len[4]} 0 0">
+                                    <joint name="joint5" axis="${cs_link_axis[5]}" />
+                                    <geom fromto="0 0 0 ${cs_link_len[5]} 0 0"
+                                        mass="${cs_link_mass[5]}" />
                                     <!-- End Effector Site -->
-                                    <site name="end_effector" pos="0 0 0" size="0.01" rgba="1 0 0 1" />
+                                    <site name="end_effector" pos="${cs_link_len[5]} 0 0"
+                                        size="0.01"
+                                        rgba="1 0 0 1" />
                                 </body>
                             </body>
@@ -68,4 +69,5 @@
     </worldbody>
     <actuator>
+        <motor name="motor0" joint="joint0" ctrllimited="true" ctrlrange="-100 100" />
         <motor name="motor1" joint="joint1" ctrllimited="true" ctrlrange="-100 100" />
         <motor name="motor2" joint="joint2" ctrllimited="true" ctrlrange="-100 100" />
@@ -73,5 +75,4 @@
         <motor name="motor4" joint="joint4" ctrllimited="true" ctrlrange="-100 100" />
         <motor name="motor5" joint="joint5" ctrllimited="true" ctrlrange="-100 100" />
-        <motor name="motor6" joint="joint6" ctrllimited="true" ctrlrange="-100 100" />
     </actuator>
     <keyframe>

Commit message: 関節の位置関係合わせた

File: test_sat.xacro (robot description, xacro)
@@ -10,5 +10,5 @@
     <default>
         <joint type="hinge" />
-        <geom type="capsule" size="0.05" rgba="0.6 0.8 1.0 1" />
+        <geom type="cylinder" size="0.05" rgba="0.6 0.8 1.0 1" />
     </default>
     <worldbody>
@@ -25,4 +25,5 @@
         <xacro:property name="cs_link_axis"
             value="${['0 0 1', '0 1 0', '0 1 0', '0 1 0', '0 0 1', '0 1 0']}" />
+        <xacro:property name="cs_link_offset" value="${[0.28, 0, 0, 0, 0, 0]}" />
         <!-- ChaserSatellite -->
         <body name="cs_base" pos="0 0 0">
@@ -31,31 +32,33 @@
                 size="${cs_base_size[0]/2} ${cs_base_size[1]/2} ${cs_base_size[2]/2}"
                 rgba="0.6 0.8 1.0 1" mass="${cs_base_mass}" />
-            <!-- Link 1 -->
-            <body name="link0" pos="0.6 0 0">
+            <!-- Link 0 -->
+            <body name="link0" pos="0 0 ${cs_base_size[2]/2}">
                 <joint name="joint0" axis="${cs_link_axis[0]}" />
-                <geom fromto="0 0 0 0 0 -${cs_link_len[0]}" mass="${cs_link_mass[0]}" />
-                <!-- Link 2 -->
-                <body name="link1" pos="0 0 -${cs_link_len[0]}">
+                <geom fromto="0 0 0 0 0 ${cs_link_len[0]}" mass="${cs_link_mass[0]}" />
+                <geom fromto="0 0 ${cs_link_len[0]} ${cs_link_offset[0]} 0 ${cs_link_len[0]}"
+                    mass="0" />
+                <!-- Link 1 -->
+                <body name="link1" pos="${cs_link_offset[0]} 0 ${cs_link_len[0]}">
                     <joint name="joint1" axis="${cs_link_axis[1]}" />
-                    <geom fromto="0 0 0 ${cs_link_len[1]} 0 0" mass="${cs_link_mass[1]}" />
-                    <!-- Link 3 -->
-                    <body name="link2" pos="${cs_link_len[1]} 0 0">
+                    <geom fromto="0 0 0 0 0 ${cs_link_len[1]}" mass="${cs_link_mass[1]}" />
+                    <!-- Link 2 -->
+                    <body name="link2" pos="0 0 ${cs_link_len[1]}">
                         <joint name="joint2" axis="${cs_link_axis[2]}" />
-                        <geom fromto="0 0 0 0 0 -${cs_link_len[2]}" mass="${cs_link_mass[2]}" />
-                        <!-- Link 4 -->
-                        <body name="link3" pos="0 0 -${cs_link_len[2]}">
+                        <geom fromto="0 0 0 0 -${cs_link_len[2]} 0" mass="${cs_link_mass[2]}" />
+                        <!-- Link 3 -->
+                        <body name="link3" pos="0 -${cs_link_len[2]} 0">
                             <joint name="joint3" axis="${cs_link_axis[3]}" />
-                            <geom fromto="0 0 0 ${cs_link_len[3]} 0 0" mass="${cs_link_mass[3]}" />
-                            <!-- Link 5 -->
-                            <body name="link4" pos="${cs_link_len[3]} 0 0">
+                            <geom fromto="0 0 0 -${cs_link_len[3]} 0 0" mass="${cs_link_mass[3]}" />
+                            <!-- Link 4 -->
+                            <body name="link4" pos="-${cs_link_len[3]} 0 0">
                                 <joint name="joint4" axis="${cs_link_axis[4]}" />
-                                <geom fromto="0 0 0 ${cs_link_len[4]} 0 0" mass="${cs_link_mass[4]}" />
-                                <!-- Link 6 -->
-                                <body name="link5" pos="${cs_link_len[4]} 0 0">
+                                <geom fromto="0 0 0 0 0 ${cs_link_len[4]}" mass="${cs_link_mass[4]}" />
+                                <!-- Link 5 -->
+                                <body name="link5" pos="0 0 ${cs_link_len[4]}">
                                     <joint name="joint5" axis="${cs_link_axis[5]}" />
-                                    <geom fromto="0 0 0 ${cs_link_len[5]} 0 0"
+                                    <geom fromto="0 0 0 0 -${cs_link_len[5]} 0"
                                         mass="${cs_link_mass[5]}" />
                                     <!-- End Effector Site -->
-                                    <site name="end_effector" pos="${cs_link_len[5]} 0 0"
+                                    <site name="end_effector" pos="0 -${cs_link_len[5]} 0"
                                         size="0.01"
                                         rgba="1 0 0 1" />
@@ -75,4 +78,10 @@
         <motor name="motor4" joint="joint4" ctrllimited="true" ctrlrange="-100 100" />
         <motor name="motor5" joint="joint5" ctrllimited="true" ctrlrange="-100 100" />
+        <position name="servo0" joint="joint0" kp="3" kv="5" />
+        <position name="servo1" joint="joint1" kp="3" kv="5" />
+        <position name="servo2" joint="joint2" kp="3" kv="5" />
+        <position name="servo3" joint="joint3" kp="3" kv="5" />
+        <position name="servo4" joint="joint4" kp="3" kv="5" />
+        <position name="servo5" joint="joint5" kp="3" kv="5" />
     </actuator>
     <keyframe>
